File: pcb/EngineMonitor.sch (KiCad schematic (older format))
At the start: 44 parts, among them K1 CONN_3, K2 CONN_3, K3 CONN_3, K4 CONN_3, P1 CONN_6, P2 CONN_6, P3 CONN_1, P4 CONN_1, P5 CONN_4, P6 CONN_4, P7 CONN_4, U1 74HC14, U2 ESP32Dev

Commit message: Redisigned board and fixed sensors
Parts:
- added D1: DIODE, Resistors_ThroughHole:Resistor_Horizontal_RM7mm, symbol DIODE
- C1, C2, C3, C4, C5, C6, R1, R10, R11, R12, R13, R14, R15, R16, R17, R18, R19, R2, R20, R21, R22, R23, R24, R25, R3, R4, R5, R6, R7, R8, R9: footprint Resistors_ThroughHole:Resistor_Horizontal_RM10mmLargePads -> Resistors_ThroughHole:Resistor_Horizontal_RM7mm
Connections:
- net 5v: now also D1.2 (K); no longer P3.1
- net DIN1: now also U1.12, U2.25 (D19); no longer U1.2, U2.8 (D25)
- net DIN2: now also U1.10, U2.24 (D18); no longer U1.4, U2.9 (D26)
- net DIN3: now also U1.8, U2.23 (D5); no longer U1.6, U2.10 (D27)
- net DIN4: now also U1.6, U2.22 (TX2); no longer U1.8, U2.11 (D11)
- net DIN5: now also U1.4, U2.21 (RX2); no longer U1.10, U2.12 (D12)
- net DIN6: now also U1.2, U2.20 (D4); no longer U1.12, U2.13 (D13)
- new net: D1.1 (A), P3.1
