File: pcb/NMEA2000Module.kicad_pcb (KiCad board)
At the start: 2 copper layers, 37 parts, among them IC1 MCP2562FD, IC2 MAX485/3485, K1 CONN_3, K2 CONN_3, K3 CONN_3, K4 CONN_3, P1 CONN_2, P10 CONN_4, P2 RS-485 A/B, P3 CAN H/L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

Commit message: New Board, i2C ADC + CAN connection
Parts:
- added P5: CONN_1, Pin_Headers:Pin_Header_Straight_1x01_Pitch2.54mm, F.Cu at (145.0, 107.5)
- K1: value CONN_3 -> 1W1
- K2: value CONN_3 -> 1W2
- K3: value CONN_3 -> 1W3
- K4: value CONN_3 -> 1W4
- P1: value CONN_2 -> PULSE_IN
- P10: value CONN_4 -> I2C3
- P6: value CONN_10 -> ADS1115
- P7: value CONN_4 -> I2C1
- P8: value CONN_4 -> I2C2
- P9: value CONN_4 -> ANALOG IN
- moved P4 104.9 mm to (156.9, 107.2)
- moved P4 103.1 mm to (144.9, 107.5)
- moved D1 80.6 mm to (143.2, 125.3), turned to 180 degrees
- moved K1 14.9 mm to (82.3, 89.5), turned to 0 degrees
- moved K4 9.92 mm to (78.6, 89.5), turned to 0 degrees
- moved R12 6.32 mm to (65.2, 96.7), turned to 90 degrees
- moved P1 6.15 mm to (138.2, 142.2)
- moved K2 5.41 mm to (74.9, 89.5), turned to 0 degrees
- moved P8 4.88 mm to (87.6, 122.5)
- moved P7 4.49 mm to (87.4, 127.0)
- moved K3 3.72 mm to (71.3, 89.5), turned to 0 degrees
- moved P10 3.06 mm to (87.4, 133.0)
Connections:
- P10 pad 1: GND -> +3.3V
- P10 pad 2: SCL -> GND
- P10 pad 3: SDA -> SCL
- P10 pad 4: +3.3V -> SDA
- P7 pad 1: GND -> +3.3V
- P7 pad 2: SCL -> GND
- P7 pad 3: SDA -> SCL
- P7 pad 4: +3.3V -> SDA
- P8 pad 1: GND -> +3.3V
- P8 pad 2: SCL -> GND
- P8 pad 3: SDA -> SCL
- P8 pad 4: +3.3V -> SDA
Routing:
- net +3.3V: track 250.6 -> 187.2 mm
- net GND: track 379.2 -> 436.1 mm
- net 5v: track 120.4 -> 76.4 mm, vias 4 -> 2
- net +5V: track 11.2 -> 23.9 mm
- net 1Wire: track 63.5 -> 72.5 mm, vias 2 -> 0
- net Net-(P1-Pad2): track 18.8 -> 11.7 mm
- net Net-(P1-Pad1): track 9.34 -> 4.97 mm
- net SCL: track 48.2 -> 50.7 mm
- net SDA: track 48.8 -> 50.7 mm
- net (no net): track 0.00 -> 0.57 mm
Other:
- board text added: "(c) Ian Boston 2020 NMEA2000 Sensor Board"
- board text removed: "(c) Ian Boston 2020 Signalk Sensor Board"
