File: pcb/NMEA2000Module.kicad_pcb (KiCad board)
At the start: 2 copper layers, 78 x 124 mm, 45 parts, among them IC1 MCP2562FD, K1 1W1, P1 PULSE_IN, P2 CONN_6, P3 TERM_R, P4 CAN, P7 I2C1, U1 74HC14, U2 ESP32Dev, U3 JDY40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

Commit message: Update to pcb to reflect prototype
Parts:
- added R5: 10K, Resistors_SMD:R_0805_HandSoldering, B.Cu at (116.7, 121.6)
Connections:
- U2 pad 7: BTENABLE -> (no net)
- U2 pad 8: (no net) -> BTENABLE
Routing:
- net 3v3: track 289.7 -> 287.2 mm
- net BTENABLE: track 28.2 -> 27.5 mm
Changed lines of the file:
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@@
 (kicad_pcb (version 4) (host pcbnew 4.0.6)
   (general
-    (links 108)
-    (no_connects 0)
+    (links 110)
+    (no_connects 1)
     (area 98.424999 55.424999 176.575001 179.575001)
     (thickness 1.6)
     (drawings 54)
-    (tracks 493)
+    (tracks 495)
     (zones 0)
-    (modules 45)
+    (modules 46)
     (nets 34)
   )
@@
     (pad 24 thru_hole oval (at 21.082 2.732 270) (size 2 3.5) (drill 1) (layers *.Cu *.Mask)
       (net 13 CAN-RX))
-    (pad 7 thru_hole oval (at 21.082 26.732 270) (size 2 3.5) (drill 1) (layers *.Cu *.Mask)
-      (net 27 BTENABLE))
+    (pad 7 thru_hole oval (at 21.082 26.732 270) (size 2 3.5) (drill 1) (layers *.Cu *.Mask))
     (pad 23 thru_hole oval (at 23.622 2.732 270) (size 2 3.5) (drill 1) (layers *.Cu *.Mask)
       (net 20 SERIALEN))
-    (pad 8 thru_hole oval (at 23.622 26.732 270) (size 2 3.5) (drill 1) (layers *.Cu *.Mask))
+    (pad 8 thru_hole oval (at 23.622 26.732 270) (size 2 3.5) (drill 1) (layers *.Cu *.Mask)
+      (net 27 BTENABLE))
     (pad 22 thru_hole oval (at 26.162 2.732 270) (size 2 3.5) (drill 1) (layers *.Cu *.Mask)
       (net 19 SERIALTX))
@@
       (scale (xyz 1 1 1))
       (rotate (xyz 0 0 90))
+    )
+  )
+  (module Resistors_SMD:R_0805_HandSoldering (layer B.Cu)
+    (at 116.7 121.6 90)
+    (descr "Resistor SMD 0805, hand soldering")
+    (tags "resistor 0805")
+    (attr smd)
+    (fp_text reference R5 (at 0 2.1 90) (layer B.SilkS)
+      (effects (font (size 1 1) (thickness 0.15)) (justify mirror))
+    )
+    (fp_text value 10K (at 0 -2.1 90) (layer B.Fab)
+      (effects (font (size 1 1) (thickness 0.15)) (justify mirror))
+    )
+    (fp_line (start -1 -0.625) (end -1 0.625) (layer B.Fab) (width 0.1))
+    (fp_line (start 1 -0.625) (end -1 -0.625) (layer B.Fab) (width 0.1))
+    (fp_line (start 1 0.625) (end 1 -0.625) (layer B.Fab) (width 0.1))
+    (fp_line (start -1 0.625) (end 1 0.625) (layer B.Fab) (width 0.1))
+    (fp_line (start -2.4 1) (end 2.4 1) (layer B.CrtYd) (width 0.05))
+    (fp_line (start -2.4 -1) (end 2.4 -1) (layer B.CrtYd) (width 0.05))
+    (fp_line (start -2.4 1) (end -2.4 -1) (layer B.CrtYd) (width 0.05))
+    (fp_line (start 2.4 1) (end 2.4 -1) (layer B.CrtYd) (width 0.05))
+    (fp_line (start 0.6 -0.875) (end -0.6 -0.875) (layer B.SilkS) (width 0.15))
+    (fp_line (start -0.6 0.875) (end 0.6 0.875) (layer B.SilkS) (width 0.15))
+    (pad 1 smd rect (at -1.35 0 90) (size 1.5 1.3) (layers B.Cu B.Paste B.Mask)
+      (net 14 3v3))
+    (pad 2 smd rect (at 1.35 0 90) (size 1.5 1.3) (layers B.Cu B.Paste B.Mask)
+      (net 27 BTENABLE))
+    (model Resistors_SMD.3dshapes/R_0805_HandSoldering.wrl
+      (at (xyz 0 0 0))
+      (scale (xyz 1 1 1))
+      (rotate (xyz 0 0 0))
     )
   )
@@
   (segment (start 157.432 95.982) (end 149.818 95.982) (width 1) (layer B.Cu) (net 13))
   (segment (start 160.03 98.58) (end 157.432 95.982) (width 1) (layer B.Cu) (net 13))
-  (segment (start 102.2 124.8) (end 102.2 126.12) (width 1) (layer B.Cu) (net 14) (status 800000))
-  (segment (start 102.2 126.12) (end 102.258 126.178) (width 1) (layer B.Cu) (net 14) (status C00000))
-  (segment (start 111.7 123.35) (end 103.65 123.35) (width 1) (layer B.Cu) (net 14) (status 400000))
+  (segment (start 116.7 122.95) (end 112.1 122.95) (width 1) (layer B.Cu) (net 14) (status C00000))
+  (segment (start 112.1 122.95) (end 111.7 123.35) (width 1) (layer B.Cu) (net 14) (status C00000))
+  (segment (start 102.2 124.8) (end 102.2 126.12) (width 1) (layer B.Cu) (net 14))
+  (segment (start 102.2 126.12) (end 102.258 126.178) (width 1) (layer B.Cu) (net 14))
+  (segment (start 111.7 123.35) (end 103.65 123.35) (width 1) (layer B.Cu) (net 14))
   (segment (start 102.2 124.8) (end 102.1 124.8) (width 1) (layer B.Cu) (net 14))
   (segment (start 103.65 123.35) (end 102.2 124.8) (width 1) (layer B.Cu) (net 14))
-  (segment (start 118.75 121.9) (end 115 121.9) (width 1) (layer B.Cu) (net 14))
   (segment (start 143.85 121.85) (end 143.5 122.2) (width 1) (layer B.Cu) (net 14))
   (via (at 143.5 122.2) (size 2) (drill 1) (layers F.Cu B.Cu) (net 14))
@@
   (segment (start 118.75 121.9) (end 119 122.15) (width 1) (layer F.Cu) (net 14))
   (via (at 118.75 121.9) (size 2) (drill 1) (layers F.Cu B.Cu) (net 14))
-  (segment (start 113.55 123.35) (end 111.7 123.35) (width 1) (layer B.Cu) (net 14) (status 800000))
-  (segment (start 115 121.9) (end 113.55 123.35) (width 1) (layer B.Cu) (net 14))
   (segment (start 108.1 140.2) (end 108.1 142) (width 1) (layer B.Cu) (net 14))
   (segment (start 100.88 141) (end 100.88 138) (width 1) (layer B.Cu) (net 14))
@@
   (segment (start 165.25 118.5) (end 165.25 120.01) (width 1) (layer B.Cu) (net 26))
   (segment (start 165.25 120.01) (end 165.29 120.05) (width 1) (layer B.Cu) (net 26))
+  (segment (start 116.8 119) (end 116.8 120.15) (width 1) (layer B.Cu) (net 27) (status C00000))
+  (segment (start 116.8 120.15) (end 116.7 120.25) (width 1) (layer B.Cu) (net 27) (status C00000))
+  (segment (start 119.2 112.1) (end 119.2 102.1) (width 1) (layer B.Cu) (net 27))
+  (segment (start 122.778 98.522) (end 125.818 98.522) (width 1) (layer B.Cu) (net 27))
+  (segment (start 119.2 102.1) (end 122.778 98.522) (width 1) (layer B.Cu) (net 27))
   (segment (start 117.9 113.4) (end 117.1 114.2) (width 1) (layer B.Cu) (net 27))
-  (segment (start 119.3 100.2) (end 119.3 112) (width 1) (layer B.Cu) (net 27))
-  (segment (start 119.3 112) (end 117.9 113.4) (width 1) (layer B.Cu) (net 27))
-  (segment (start 123.518 95.982) (end 119.3 100.2) (width 1) (layer B.Cu) (net 27))
-  (segment (start 125.818 95.982) (end 123.518 95.982) (width 1) (layer B.Cu) (net 27))
-  (segment (start 116.7 114.6) (end 116.7 118.9) (width 1) (layer B.Cu) (net 27) (status 800000))
+  (segment (start 119.3 112) (end 119.2 112.1) (width 1) (layer B.Cu) (net 27))
+  (segment (start 119.2 112.1) (end 117.9 113.4) (width 1) (layer B.Cu) (net 27))
+  (segment (start 116.7 114.6) (end 116.7 118.9) (width 1) (layer B.Cu) (net 27))
   (segment (start 117.1 114.2) (end 116.7 114.6) (width 1) (layer B.Cu) (net 27))
-  (segment (start 116.7 118.9) (end 116.8 119) (width 1) (layer B.Cu) (net 27) (status C00000))
+  (segment (start 116.7 118.9) (end 116.8 119) (width 1) (layer B.Cu) (net 27))
   (segment (start 146.95 161.2) (end 146.95 164.71) (width 1) (layer B.Cu) (net 28))
   (segment (start 146.95 164.71) (end 147.16 164.92) (width 1) (layer B.Cu) (net 28))
@@
   (segment (start 109.247 117.352) (end 109.247 115.738) (width 1) (layer B.Cu) (net 32) (status 30))
   (segment (start 109.247 118.933) (end 109.18 119) (width 1) (layer B.Cu) (net 32))
-  (segment (start 111.7 120.65) (end 111.7 119.02) (width 1) (layer B.Cu) (net 33) (status C00000))
-  (segment (start 111.7 119.02) (end 111.72 119) (width 1) (layer B.Cu) (net 33) (status C00000))
+  (segment (start 111.7 120.65) (end 111.7 119.02) (width 1) (layer B.Cu) (net 33))
+  (segment (start 111.7 119.02) (end 111.72 119) (width 1) (layer B.Cu) (net 33))
   (segment (start 111.787 118.933) (end 111.787 117.352) (width 1) (layer B.Cu) (net 33))
   (segment (start 111.787 117.352) (end 111.787 115.738) (width 1) (layer B.Cu) (net 33) (status 30))
@@
     (connect_pads yes (clearance 1))
     (min_thickness 1)
-    (fill (arc_segments 16) (thermal_gap 0.508) (thermal_bridge_width 1.1))
+    (fill yes (arc_segments 16) (thermal_gap 0.508) (thermal_bridge_width 1.1))
     (polygon
       (pts
